Commit message: added full project scenes and description

File: models/descriptions/robots/mobile/tri_homecart/homecart_bimanual.urdf (robot description, URDF)
Before this commit: robot homecart_bimanual, 10 links, 9 joints
Joints:
- removed joint homecart_base_link
- added joint homecart_base_joint: type fixed, parent homecart_base_link, child homecart_baseplate_link, origin xyz=0.2775 0 0 rpy=0 0 0
